File: SpeakersShiftReg.kicad_pcb (KiCad board)
At the start: 2 copper layers, 27 parts, among them J1 CONN, J10 Conn_01x08_Male, J11 Conn_01x08_Male, J12 Conn_01x08_Male, J13 Conn_01x08_Male, J2 CONN, J3 CONN, J4 CONN, J5 CONN, J6 CONN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

Commit message: added silk, ready for traces
Parts:
- moved U2 2.07 mm to (34.9, 40.4)
- moved RN1 1.42 mm to (29.3, 40.4)
- moved U1 1.42 mm to (29.3, 53.2)
- moved H3 0.63 mm to (2.54, 50.8)
- moved R1 0.51 mm to (0.00, 41.7)
- moved R2 0.51 mm to (7.62, 59.9)
Connections:
- J10 pad 2: S_CLK -> CS
- J10 pad 3: CS -> S_CLK
Other:
- board text added: "5V"
- board text added: "CARRY"
- board text added: "CLK"
- board text added: "CLR"
- board text added: "CS"
- board text added: "DAT"
- board text added: "EN"
- board text added: "GND"
- board text added: "VDD"
Changed lines of the file:
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@@
   (general
     (thickness 1.6)
-    (drawings 15)
+    (drawings 48)
     (tracks 0)
     (zones 0)
@@
     (45 Margin user)
     (46 B.CrtYd user)
-    (47 F.CrtYd user hide)
+    (47 F.CrtYd user)
     (48 B.Fab user)
-    (49 F.Fab user hide)
+    (49 F.Fab user)
   )
   (setup
-    (last_trace_width 0.25)
+    (last_trace_width 1.25)
+    (user_trace_width 0.5)
+    (user_trace_width 1)
+    (user_trace_width 1.25)
     (trace_clearance 0.2)
     (zone_clearance 0.508)
@@
   )
   (module HammerheadAudio:M3_MOUNT (layer F.Cu)
-    (at 2.54 50.165)
+    (at 2.54 50.8)
     (descr "STANDOFF (#4 SCREW)")
     (tags "STANDOFF (#4 SCREW)")
@@
   )
   (module HammerheadAudio:R_THT_P7.62 (layer F.Cu)
-    (at -0.508 41.656)
+    (at 0 41.656)
     (descr "Resistor, Axial_DIN0207 series, Axial, Horizontal, pin pitch=7.62mm, 0.25W = 1/4W, length*diameter=6.3*2.5mm^2, http://cdn-reichelt.de/documents/datenblatt/B400/1_4W%23YAG.pdf")
     (tags "Resistor Axial_DIN0207 series Axial Horizontal pin pitch 7.62mm 0.25W = 1/4W length 6.3mm diameter 2.5mm")
@@
   )
   (module HammerheadAudio:R_THT_P7.62 (layer F.Cu)
-    (at 7.112 59.944 180)
+    (at 7.62 59.944 180)
     (descr "Resistor, Axial_DIN0207 series, Axial, Horizontal, pin pitch=7.62mm, 0.25W = 1/4W, length*diameter=6.3*2.5mm^2, http://cdn-reichelt.de/documents/datenblatt/B400/1_4W%23YAG.pdf")
     (tags "Resistor Axial_DIN0207 series Axial Horizontal pin pitch 7.62mm 0.25W = 1/4W length 6.3mm diameter 2.5mm")
@@
   )
   (module Package_DIP:DIP-16_W7.62mm_Socket (layer F.Cu)
-    (at 28.067 39.751 270)
+    (at 29.337 40.386 270)
     (descr "16-lead though-hole mounted DIP package, row spacing 7.62 mm (300 mils), Socket")
     (tags "THT DIP DIL PDIP 2.54mm 7.62mm 300mil Socket")
@@
   )
   (module Package_DIP:DIP-16_W7.62mm_Socket (layer F.Cu)
-    (at 28.067 52.578 270)
+    (at 29.337 53.213 270)
     (descr "16-lead though-hole mounted DIP package, row spacing 7.62 mm (300 mils), Socket")
     (tags "THT DIP DIL PDIP 2.54mm 7.62mm 300mil Socket")
@@
   )
   (module Package_DIP:DIP-18_W7.62mm_Socket (layer F.Cu)
-    (at 32.9565 39.8145)
+    (at 34.925 40.4495)
     (descr "18-lead though-hole mounted DIP package, row spacing 7.62 mm (300 mils), Socket")
     (tags "THT DIP DIL PDIP 2.54mm 7.62mm 300mil Socket")
@@
       (net 25 S_DAT))
     (pad 2 thru_hole oval (at 0 2.54 180) (size 1.7 1.7) (drill 1) (layers *.Cu *.Mask)
+      (net 24 CS))
+    (pad 3 thru_hole oval (at 0 5.08 180) (size 1.7 1.7) (drill 1) (layers *.Cu *.Mask)
       (net 23 S_CLK))
-    (pad 3 thru_hole oval (at 0 5.08 180) (size 1.7 1.7) (drill 1) (layers *.Cu *.Mask)
-      (net 24 CS))
     (pad 4 thru_hole oval (at 0 7.62 180) (size 1.7 1.7) (drill 1) (layers *.Cu *.Mask)
       (net 1 GND))
@@
     )
   )
+  (gr_line (start 48.514 38.1) (end 49.022 38.1) (layer F.SilkS) (width 0.12))
+  (gr_line (start 48.514 30.988) (end 48.514 38.1) (layer F.SilkS) (width 0.12))
+  (gr_line (start 48.514 20.32) (end 49.022 20.32) (layer F.SilkS) (width 0.12))
+  (gr_line (start 48.514 27.432) (end 48.514 20.32) (layer F.SilkS) (width 0.12))
+  (gr_line (start 2.286 20.32) (end 2.286 22.352) (layer F.SilkS) (width 0.12))
+  (gr_line (start 1.778 20.32) (end 2.286 20.32) (layer F.SilkS) (width 0.12))
+  (gr_line (start 2.286 27.94) (end 2.286 25.908) (layer F.SilkS) (width 0.12))
+  (gr_line (start 1.778 27.94) (end 2.286 27.94) (layer F.SilkS) (width 0.12))
+  (gr_line (start 2.286 38.1) (end 1.778 38.1) (layer F.SilkS) (width 0.12))
+  (gr_line (start 2.286 35.56) (end 2.286 38.1) (layer F.SilkS) (width 0.12))
+  (gr_line (start 2.286 30.48) (end 2.286 33.02) (layer F.SilkS) (width 0.12))
+  (gr_line (start 1.778 30.48) (end 2.286 30.48) (layer F.SilkS) (width 0.12))
+  (gr_text GND (at 2.286 24.13 90) (layer F.SilkS)
+    (effects (font (size 1 1) (thickness 0.15)))
+  )
+  (gr_text 5V (at 2.286 34.29 90) (layer F.SilkS)
+    (effects (font (size 1 1) (thickness 0.15)))
+  )
+  (gr_text VDD (at 48.514 29.21 90) (layer F.SilkS)
+    (effects (font (size 1 1) (thickness 0.15)))
+  )
+  (gr_line (start 48.514 81.28) (end 49.022 81.28) (layer F.SilkS) (width 0.12))
+  (gr_line (start 48.514 74.168) (end 48.514 81.28) (layer F.SilkS) (width 0.12))
+  (gr_line (start 48.514 63.5) (end 49.022 63.5) (layer F.SilkS) (width 0.12))
+  (gr_line (start 48.514 70.612) (end 48.514 63.5) (layer F.SilkS) (width 0.12))
+  (gr_text GND (at 48.514 72.39 90) (layer F.SilkS)
+    (effects (font (size 1 1) (thickness 0.15)))
+  )
+  (gr_text CARRY (at 1.524 63.5) (layer F.SilkS)
+    (effects (font (size 0.5 0.5) (thickness 0.1)) (justify left))
+  )
+  (gr_text EN (at 1.524 68.58) (layer F.SilkS)
+    (effects (font (size 0.5 0.5) (thickness 0.1)) (justify left))
+  )
+  (gr_text GND (at 1.524 66.04) (layer F.SilkS)
+    (effects (font (size 0.5 0.5) (thickness 0.1)) (justify left))
+  )
+  (gr_text GND (at 1.524 73.66) (layer F.SilkS)
+    (effects (font (size 0.5 0.5) (thickness 0.1)) (justify left))
+  )
+  (gr_text CLR (at 1.524 71.12) (layer F.SilkS)
+    (effects (font (size 0.5 0.5) (thickness 0.1)) (justify left))
+  )
+  (gr_text CLK (at 1.524 76.2) (layer F.SilkS)
+    (effects (font (size 0.5 0.5) (thickness 0.1)) (justify left))
+  )
+  (gr_text CS (at 1.524 78.74) (layer F.SilkS)
+    (effects (font (size 0.5 0.5) (thickness 0.1)) (justify left))
+  )
+  (gr_text DAT (at 1.524 81.28) (layer F.SilkS)
+    (effects (font (size 0.5 0.5) (thickness 0.1)) (justify left))
+  )
+  (dimension 12.7 (width 0.15) (layer Cmts.User)
+    (gr_text "12.700 mm" (at -21.62 44.45 270) (layer Cmts.User)
+      (effects (font (size 1 1) (thickness 0.15)))
+    )
+    (feature1 (pts (xy 0 50.8) (xy -20.906421 50.8)))
+    (feature2 (pts (xy 0 38.1) (xy -20.906421 38.1)))
+    (crossbar (pts (xy -20.32 38.1) (xy -20.32 50.8)))
+    (arrow1a (pts (xy -20.32 50.8) (xy -20.906421 49.673496)))
+    (arrow1b (pts (xy -20.32 50.8) (xy -19.733579 49.673496)))
+    (arrow2a (pts (xy -20.32 38.1) (xy -20.906421 39.226504)))
+    (arrow2b (pts (xy -20.32 38.1) (xy -19.733579 39.226504)))
+  )
+  (dimension 25.4 (width 0.15) (layer Cmts.User)
+    (gr_text "25.400 mm" (at -8.285 50.8 270) (layer Cmts.User)
+      (effects (font (size 1 1) (thickness 0.15)))
+    )
+    (feature1 (pts (xy 0 63.5) (xy -7.571421 63.5)))
+    (feature2 (pts (xy 0 38.1) (xy -7.571421 38.1)))
+    (crossbar (pts (xy -6.985 38.1) (xy -6.985 63.5)))
+    (arrow1a (pts (xy -6.985 63.5) (xy -7.571421 62.373496)))
+    (arrow1b (pts (xy -6.985 63.5) (xy -6.398579 62.373496)))
+    (arrow2a (pts (xy -6.985 38.1) (xy -7.571421 39.226504)))
+    (arrow2b (pts (xy -6.985 38.1) (xy -6.398579 39.226504)))
+  )
+  (dimension 25.4 (width 0.15) (layer Cmts.User)
+    (gr_text "25.400 mm" (at 66.705 50.8 270) (layer Cmts.User)
+      (effects (font (size 1 1) (thickness 0.15)))
+    )
+    (feature1 (pts (xy 50.8 63.5) (xy 65.991421 63.5)))
+    (feature2 (pts (xy 50.8 38.1) (xy 65.991421 38.1)))
+    (crossbar (pts (xy 65.405 38.1) (xy 65.405 63.5)))
+    (arrow1a (pts (xy 65.405 63.5) (xy 64.818579 62.373496)))
+    (arrow1b (pts (xy 65.405 63.5) (xy 65.991421 62.373496)))
+    (arrow2a (pts (xy 65.405 38.1) (xy 64.818579 39.226504)))
+    (arrow2b (pts (xy 65.405 38.1) (xy 65.991421 39.226504)))
+  )
+  (dimension 15.8115 (width 0.15) (layer Cmts.User)
+    (gr_text "15.812 mm" (at 6.447 42.83075 270) (layer Cmts.User)
+      (effects (font (size 1 1) (thickness 0.15)))
+    )
+    (feature1 (pts (xy 19.685 50.7365) (xy 7.160579 50.7365)))
+    (feature2 (pts (xy 19.685 34.925) (xy 7.160579 34.925)))
+    (crossbar (pts (xy 7.747 34.925) (xy 7.747 50.7365)))
+    (arrow1a (pts (xy 7.747 50.7365) (xy 7.160579 49.609996)))
+    (arrow1b (pts (xy 7.747 50.7365) (xy 8.333421 49.609996)))
+    (arrow2a (pts (xy 7.747 34.925) (xy 7.160579 36.051504)))
+    (arrow2b (pts (xy 7.747 34.925) (xy 8.333421 36.051504)))
+  )
+  (dimension 31.623 (width 0.15) (layer Cmts.User)
+    (gr_text "31.623 mm" (at 20.985 50.7365 90) (layer Cmts.User)
+      (effects (font (size 1 1) (thickness 0.15)))
+    )
+    (feature1 (pts (xy 19.685 34.925) (xy 20.271421 34.925)))
+    (feature2 (pts (xy 19.685 66.548) (xy 20.271421 66.548)))
+    (crossbar (pts (xy 19.685 66.548) (xy 19.685 34.925)))
+    (arrow1a (pts (xy 19.685 34.925) (xy 20.271421 36.051504)))
+    (arrow1b (pts (xy 19.685 34.925) (xy 19.098579 36.051504)))
+    (arrow2a (pts (xy 19.685 66.548) (xy 20.271421 65.421496)))
+    (arrow2b (pts (xy 19.685 66.548) (xy 19.098579 65.421496)))
+  )
   (dimension 60.96 (width 0.15) (layer Cmts.User)

Commit message: commit before trying thing
Routing:
- net VDD: track 0.00 -> 97.8 mm
- net Net-(D8-Pad2): track 0.00 -> 85.6 mm
- net Net-(D7-Pad2): track 0.00 -> 73.5 mm
- net Net-(D6-Pad2): track 0.00 -> 63.4 mm
- net +5V: track 0.00 -> 56.8 mm
- net Net-(D5-Pad2): track 0.00 -> 52.8 mm
- net CLEAR: track 0.00 -> 44.0 mm
- net QA: track 0.00 -> 40.3 mm
- net S_DAT: track 0.00 -> 40.2 mm
- net CS: track 0.00 -> 31.8 mm
- net QH: track 0.00 -> 29.2 mm
- net ENABLE: track 0.00 -> 28.6 mm
- net S_CLK: track 0.00 -> 27.1 mm
- net Net-(D4-Pad2): track 0.00 -> 26.4 mm
- net QG: track 0.00 -> 25.9 mm
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Other:
- board outline added: 55.9 x 66 mm
- board text added: "+"
- board text added: "-"

Commit message: finish layout
Parts:
- added C1: 0.1uf, Capacitor_THT:C_Disc_D3.0mm_W2.0mm_P2.50mm, F.Cu at (6.35, 44.2)
- added C2: 10uf, Capacitor_THT:CP_Radial_D5.0mm_P2.00mm, F.Cu at (1.27, 44.3)
- added C3: 10uf, Capacitor_THT:CP_Radial_D5.0mm_P2.00mm, F.Cu at (50.8, 37.5)
- added C4: 10uf, Capacitor_THT:CP_Radial_D5.0mm_P2.00mm, F.Cu at (50.8, 64.0)
- added HHLogo_11.5mm: Val**, HammerheadAudio:HHLOGO_11mm, B.Cu at (30.7, 68.1)
- J10, J11, J12, J13: footprint Connector_PinSocket_2.54mm:PinSocket_1x08_P2.54mm_Vertical -> Connector_PinSocket_2.54mm:PinSocket_1x06_P2.54mm_Vertical
- moved H3 2.54 mm to (2.54, 53.3)
- moved R1 1.02 mm to (0.00, 40.6)
- moved R2 0.76 mm to (7.62, 60.7)
- moved D1 0.25 mm to (8.26, 35.9)
- moved D2 0.25 mm to (19.7, 35.9)
- moved D3 0.25 mm to (31.1, 35.9)
- moved D4 0.25 mm to (42.5, 35.9)
- moved D5 0.13 mm to (42.5, 65.4)
- moved D6 0.13 mm to (31.1, 65.4)
- moved D7 0.13 mm to (19.7, 65.4)
- moved D8 0.13 mm to (8.26, 65.4)
Connections:
- J10 pad 4: GND -> CLEAR
- J10 pad 5: CLEAR -> ENABLE
- J10 pad 6: ENABLE -> CARRY_OUT
- J13 pad 4: GND -> +5V
Routing:
- net VDD: track 97.8 -> 188.8 mm
- net O8: track 6.32 -> 62.8 mm
- net O1: track 7.11 -> 60.4 mm
- net O2: track 6.32 -> 43.1 mm
- net O3: track 6.32 -> 42.7 mm
- net O7: track 6.32 -> 42.6 mm
- net O6: track 6.32 -> 42.1 mm
- net O4: track 6.32 -> 34.8 mm
- net O5: track 6.32 -> 34.5 mm
- net +5V: track 56.8 -> 70.7 mm
- net Net-(D6-Pad2): track 63.4 -> 57.0 mm
- net ENABLE: track 28.6 -> 33.2 mm
- net Net-(D7-Pad2): track 73.5 -> 69.4 mm
- net Net-(D8-Pad2): track 85.6 -> 82.0 mm
- net S_CLK: track 27.1 -> 29.5 mm
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- added copper zone on F.Cu, net GND
Other:
- board text added: "HAMMERHEAD AUDIO - SHIFT DRIVER V1.0 - E. PALAIMA"
- board text added: "J1"
- board text added: "J2"
- board text added: "J3"
- board text added: "J4"
- board text added: "J5"
- board text added: "J6"
- board text added: "J7"
- board text added: "J8"
- board text added: "SHIFT DRIVER V0.1 HHAUDIO 2020 E. PALAIMA"

Commit message: finished layout
Other:
- board text added: "O1"
- board text added: "O2"
- board text added: "O3"
- board text added: "O4"
- board text added: "O5"
- board text added: "O6"
- board text added: "O7"
- board text added: "O8"
Changed lines of the file:
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@@
   (general
     (thickness 1.6)
-    (drawings 96)
+    (drawings 112)
     (tracks 318)
     (zones 0)
@@
     )
   )
+  (dimension 2.54 (width 0.15) (layer Cmts.User)
+    (gr_text "2.540 mm" (at 52.07 -0.03) (layer Cmts.User)
+      (effects (font (size 1 1) (thickness 0.15)))
+    )
+    (feature1 (pts (xy 53.34 41.91) (xy 53.34 0.683579)))
+    (feature2 (pts (xy 50.8 41.91) (xy 50.8 0.683579)))
+    (crossbar (pts (xy 50.8 1.27) (xy 53.34 1.27)))
+    (arrow1a (pts (xy 53.34 1.27) (xy 52.213496 1.856421)))
+    (arrow1b (pts (xy 53.34 1.27) (xy 52.213496 0.683579)))
+    (arrow2a (pts (xy 50.8 1.27) (xy 51.926504 1.856421)))
+    (arrow2b (pts (xy 50.8 1.27) (xy 51.926504 0.683579)))
+  )
+  (dimension 24.13 (width 0.15) (layer Cmts.User)
+    (gr_text "24.130 mm" (at 77.5 29.845 90) (layer Cmts.User)
+      (effects (font (size 1 1) (thickness 0.15)))
+    )
+    (feature1 (pts (xy 50.8 17.78) (xy 76.786421 17.78)))
+    (feature2 (pts (xy 50.8 41.91) (xy 76.786421 41.91)))
+    (crossbar (pts (xy 76.2 41.91) (xy 76.2 17.78)))
+    (arrow1a (pts (xy 76.2 17.78) (xy 76.786421 18.906504)))
+    (arrow1b (pts (xy 76.2 17.78) (xy 75.613579 18.906504)))
+    (arrow2a (pts (xy 76.2 41.91) (xy 76.786421 40.783496)))
+    (arrow2b (pts (xy 76.2 41.91) (xy 75.613579 40.783496)))
+  )
+  (dimension 8.89 (width 0.15) (layer Cmts.User)
+    (gr_text "8.890 mm" (at 78.77 46.355 90) (layer Cmts.User)
+      (effects (font (size 1 1) (thickness 0.15)))
+    )
+    (feature1 (pts (xy 50.8 41.91) (xy 78.056421 41.91)))
+    (feature2 (pts (xy 50.8 50.8) (xy 78.056421 50.8)))
+    (crossbar (pts (xy 77.47 50.8) (xy 77.47 41.91)))
+    (arrow1a (pts (xy 77.47 41.91) (xy 78.056421 43.036504)))
+    (arrow1b (pts (xy 77.47 41.91) (xy 76.883579 43.036504)))
+    (arrow2a (pts (xy 77.47 50.8) (xy 78.056421 49.673496)))
+    (arrow2b (pts (xy 77.47 50.8) (xy 76.883579 49.673496)))
+  )
+  (dimension 33.02 (width 0.15) (layer Cmts.User)
+    (gr_text "33.020 mm" (at 87.66 34.29 90) (layer Cmts.User)
+      (effects (font (size 1 1) (thickness 0.15)))
+    )
+    (feature1 (pts (xy 50.8 17.78) (xy 86.946421 17.78)))
+    (feature2 (pts (xy 50.8 50.8) (xy 86.946421 50.8)))
+    (crossbar (pts (xy 86.36 50.8) (xy 86.36 17.78)))
+    (arrow1a (pts (xy 86.36 17.78) (xy 86.946421 18.906504)))
+    (arrow1b (pts (xy 86.36 17.78) (xy 85.773579 18.906504)))
+    (arrow2a (pts (xy 86.36 50.8) (xy 86.946421 49.673496)))
+    (arrow2b (pts (xy 86.36 50.8) (xy 85.773579 49.673496)))
+  )
+  (gr_text O7 (at 44.45 57.15) (layer F.SilkS)
+    (effects (font (size 1 1) (thickness 0.15)) (justify left))
+  )
+  (gr_text O8 (at 44.45 59.69) (layer F.SilkS)
+    (effects (font (size 1 1) (thickness 0.15)) (justify left))
+  )
+  (gr_text O6 (at 44.45 54.61) (layer F.SilkS)
+    (effects (font (size 1 1) (thickness 0.15)) (justify left))
+  )
+  (gr_text O5 (at 44.45 52.07) (layer F.SilkS)
+    (effects (font (size 1 1) (thickness 0.15)) (justify left))
+  )
+  (gr_text O4 (at 44.45 49.53) (layer F.SilkS)
+    (effects (font (size 1 1) (thickness 0.15)) (justify left))
+  )
+  (gr_text O3 (at 44.45 46.99) (layer F.SilkS)
+    (effects (font (size 1 1) (thickness 0.15)) (justify left))
+  )
+  (gr_text O2 (at 44.45 44.45) (layer F.SilkS)
+    (effects (font (size 1 1) (thickness 0.15)) (justify left))
+  )
+  (gr_text O1 (at 44.45 41.91) (layer F.SilkS)
+    (effects (font (size 1 1) (thickness 0.15)) (justify left))
+  )
+  (gr_text - (at 46.736 61.468 180) (layer F.SilkS)
+    (effects (font (size 1 1) (thickness 0.15)))
+  )
+  (gr_text + (at 52.451 61.468 180) (layer F.SilkS)
+    (effects (font (size 1 1) (thickness 0.15)))
+  )
+  (gr_text - (at 46.736 40.259 180) (layer F.SilkS)
+    (effects (font (size 1 1) (thickness 0.15)))
+  )
+  (gr_text + (at 52.451 40.259 180) (layer F.SilkS)
+    (effects (font (size 1 1) (thickness 0.15)))
+  )
   (gr_text "HAMMERHEAD AUDIO - SHIFT DRIVER V1.0 - E. PALAIMA" (at 25.4 81.28) (layer B.SilkS)
